Commit message: modified some urdf files, yamle files and launch files. Still not displaying camera and robot in rviz

File: industrial_extrinsic_cal/urdf/r430_def_macro.xacro (robot description, xacro)
@@ -28,4 +28,6 @@
   <!-- starting here is his macro !!!!!!!!!!!!!!!!!!!!!!!!!!!!!!!!!!!!!!!!!!!!!!!!!!!!!! -->
   <xacro:macro name="sensor_r430" params="parent_link prefix *origin">
+    <!-- links: one for the optical frame and one for defining the link geometry -->
+    <link name="${prefix}"/>
     <material name="${prefix}_aluminum">
       <color rgba="0.5 0.5 0.5 1"/>

File: industrial_extrinsic_cal/urdf/ur10.gazebo.xacro (robot description, xacro)
@@ -1,4 +1,4 @@
 <?xml version="1.0"?>
-<robot xmlns:xacro="http://www.ros.org/wiki/xacro">
+<robot xmlns:xacro="http://ros.org/wiki/xacro">
   <xacro:macro name="ur10_arm_gazebo" params="prefix">
     <!-- nothing to do here at the moment -->

File: industrial_extrinsic_cal/urdf/ur10.transmission.xacro (robot description, xacro)
@@ -1,4 +1,4 @@
 <?xml version="1.0"?>
-<robot xmlns:xacro="http://www.ros.org/wiki/xacro">
+<robot xmlns:xacro="http://ros.org/wiki/xacro">
   <xacro:macro name="ur10_arm_transmission" params="prefix">
     <transmission name="${prefix}shoulder_pan_trans">

File: industrial_extrinsic_cal/urdf/ur10_macro.xacro (robot description, xacro)
@@ -1,4 +1,4 @@
 <?xml version="1.0"?>
-<robot xmlns:xacro="http://www.ros.org/wiki/xacro">
+<robot xmlns:xacro="http://ros.org/wiki/xacro">
 <!--
   Author: Kelsey Hawkins
@@ -7,5 +7,5 @@
   <xacro:include filename="$(find industrial_extrinsic_cal)/urdf/ur10.transmission.xacro" />
   <xacro:include filename="$(find industrial_extrinsic_cal)/urdf/ur10.gazebo.xacro" />
-  <xacro:property name="pi" value="3.14159265" />
+  <!-- <xacro:property name="pi" value="3.14159265" /> -->
   <!-- Inertia parameters -->
   <xacro:property name="base_mass" value="4.0" />  <!-- This mass might be incorrect -->

File: industrial_extrinsic_cal/urdf/ur10_real_sense_target.xacro (robot description, xacro)
@@ -3,5 +3,6 @@
   <xacro:include filename="$(find industrial_extrinsic_cal)/urdf/ur10_macro.xacro"/>
   <xacro:include filename="$(find industrial_extrinsic_cal)/urdf/calibration_transform_macro.xacro"/>
-  <xacro:include filename="$(find industrial_extrinsic_cal)/urdf/_r430.urdf.xacro"/>
+  <xacro:include filename="$(find industrial_extrinsic_cal)/urdf/r430_def_macro.xacro"/>
+  <xacro:include filename="$(find industrial_extrinsic_cal)/urdf/ifm_cal_macro.xacro"/>
   <link name="world"/>
   <link name="tsdf_frame"/>
@@ -12,5 +13,5 @@
     <origin rpy="0 0 0" xyz="0 0 0"/>
   </joint>
-  <xacro:ur10_robot prefix=""/>
+  <xacro:ur10_robot prefix="" joint_limited="true"/>
   <!-- attach robot to world -->
   <joint name="world_to_robot" type="fixed">
@@ -48,11 +49,13 @@
          basler1_yaw_joint
          basler1_pitch_joint
-         basler1_roll_joint    -->
-      <xacro:basler_sensor_definitions prefix="basler1" parent_link="tool0"/>
-      <xacro:sensor_r430 parent_link="tool0" prefix="r430_1">
-        <origin xyz="0 0 0" rpy="0 0 0"/>
-      </xacor:sensor_r430>
-  <!-- add an ifm camera attached to the wrist -->
-  <!--This adds the following mutable joint states, add them to the mutable joint states yaml file and run the node
+         basler1_roll_joint
+  <xacro:basler_sensor_definitions prefix="basler1" parent_link="tool0"/>
+  -->
+  <!-- add real sense r430 to the wrist -->
+  <xacro:sensor_r430 prefix="r430_1" parent_link="tool0">
+        <origin xyz="0 0 0" rpy="0 0 0" />
+  </xacro:sensor_r430>
+  <!-- add an ifm camera attached to the wrist
+      This adds the following mutable joint states, add them to the mutable joint states yaml file and run the node
       ifm_x_joint
       ifm_y_joint
@@ -60,6 +63,7 @@
       ifm_yaw_joint
       ifm_pitch_joint
-      ifm_roll_joint      -->
-      <xacro:ifm_sensor_definitions prefix="ifm" parent_link="tool0"/>
+      ifm_roll_joint
+   -->
+  <xacro:ifm_sensor_definitions prefix="ifm" parent_link="tool0"/>
   <!-- add an asus camera attached to the wrist -->
   <!--This adds the following mutable joint states, add them to the mutable joint states yaml file and run the node
